Commit message: UPDATE: refactor code

File: src/robot_core/model/lidar.xacro (robot description, xacro)
@@ -2,7 +2,7 @@
 <robot xmlns:xacro="http://www.ros.org/wiki/xacro">
   <joint name="laser_joint" type="fixed">
-    <parent link="chassis"/>
+    <parent link="base_link"/>
     <child link="laser_frame"/>
-    <origin xyz="0.09 0 0.18" rpy="0 0 0"/>
+    <origin xyz="0 0 0.18" rpy="0 0 0"/>
   </joint>
   <link name="laser_frame">
@@ -46,5 +46,5 @@
         </scan>
         <range>
-          <min>0.3</min>
+          <min>0.15</min>
           <max>12</max>
         </range>

File: src/robot_core/model/robot_core.xacro (robot description, xacro)
@@ -19,6 +19,13 @@
     <color rgba="1 0 0 1"/>
   </material>
-  <!-- BASE -->
+  <!-- BASE LINK -->
   <link name="base_link"></link>
+  <!-- BASE FOOTPRINT -->
+  <joint name="base_footprint_joint" type="fixed">
+    <parent link="base_link"/>
+    <child link="base_footprint"/>
+    <origin xyz="0 0 0" rpy="0 0 0"/>
+  </joint>
+  <link name="base_footprint"></link>
   <!-- CHASSIS -->
   <joint name="chassis_joint" type="fixed">
@@ -49,5 +56,5 @@
     <parent link="base_link"/>
     <child link="left_wheel"/>
-    <origin xyz="0 0.11 0" rpy="-${pi/2} 0 0"/>
+    <origin xyz="-0.04 0.11 0" rpy="-${pi/2} 0 0"/>
     <axis xyz="0 0 1"/>
   </joint>
@@ -71,5 +78,5 @@
     <parent link="base_link"/>
     <child link="right_wheel"/>
-    <origin xyz="0 -0.11 0" rpy="${pi/2} 0 0"/>
+    <origin xyz="-0.04 -0.11 0" rpy="${pi/2} 0 0"/>
     <axis xyz="0 0 -1"/>
   </joint>
